File: untitled.sch (EAGLE design)
At the start: 22 parts, among them IC2 STM32F030C8T, U1 GY-521MPU6050, U2 RFM69CW

Commit message: Fix usasrt/i2c pins
Parts:
- removed PAD13, PAD14: (no value), wirepad:SMD2
- removed R2: (no value), rcl:R-EU_M1206
- removed U1: GY-521MPU6050, gy-521:GY-521MPU6050
- added C2: (no value), rcl:C-EUC1206
- added IC1: TPS77015, texas:TPS77015
- added R3, R4: (no value), rcl:R-EU_M0805
Connections:
- removed net N$10: IC2MCU.BOOT0, PAD13.P, R2.1
- new net N$12: IC1.!EN, IC1.IN, PAD12.P
- new net N$14: IC1.NC/FB, R3.1, R4.2
- net GND: now also C2.2, IC1.GND, IC2MCU.BOOT0, R4.1; no longer PAD14.P
- net N$9: now also IC2MCU.PA10; no longer IC2MCU.PA8
- net VCC: now also C2.1, IC1.OUT, R3.2; no longer PAD12.P, R2.2
Other:
- moved on the sheet: PAD11, PAD12, PAD4, PAD6
Changed lines of the file:
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@@
 <part name="SUPPLY5" library="supply2" deviceset="VCC" device=""/>
 <part name="GND5" library="supply1" deviceset="GND" device=""/>
-<part name="SUPPLY6" library="supply2" deviceset="VCC" device=""/>
 <part name="SUPPLY7" library="supply2" deviceset="VCC" device=""/>
-<part name="U1" library="gy-521" deviceset="GY-521" device="MPU6050"/>
-<part name="R2" library="rcl" deviceset="R-EU_" device="M1206"/>
 <part name="GND6" library="supply1" deviceset="GND" device=""/>
 <part name="SUPPLY8" library="supply2" deviceset="VCC" device=""/>
@@
 <part name="PAD11" library="wirepad" deviceset="SMD2" device=""/>
 <part name="PAD12" library="wirepad" deviceset="SMD2" device=""/>
-<part name="PAD13" library="wirepad" deviceset="SMD2" device=""/>
-<part name="PAD14" library="wirepad" deviceset="SMD2" device=""/>
 <part name="TP2" library="testpad" deviceset="TPSQ" device="TP20SQ"/>
 <part name="TP1" library="testpad" deviceset="TPSQ" device="TP20SQ"/>
+<part name="IC1" library="texas" deviceset="TPS770*" device="" technology="15"/>
+<part name="R3" library="rcl" deviceset="R-EU_" device="M0805"/>
+<part name="R4" library="rcl" deviceset="R-EU_" device="M0805"/>
+<part name="GND8" library="supply1" deviceset="GND" device=""/>
+<part name="C2" library="rcl" deviceset="C-EU" device="C1206"/>
 </parts>
 <sheets>
@@
 <instance part="GND2" gate="1" x="109.22" y="124.46"/>
 <instance part="SUPPLY5" gate="G$1" x="109.22" y="147.32"/>
-<instance part="GND5" gate="1" x="17.78" y="66.04"/>
-<instance part="SUPPLY6" gate="G$1" x="-15.24" y="76.2"/>
+<instance part="GND5" gate="1" x="7.62" y="68.58"/>
 <instance part="SUPPLY7" gate="G$1" x="129.54" y="73.66"/>
-<instance part="U1" gate="G$1" x="116.84" y="190.5" rot="R90"/>
-<instance part="R2" gate="G$1" x="-5.08" y="73.66" rot="R180"/>
-<instance part="GND6" gate="1" x="-15.24" y="45.72" rot="R90"/>
-<instance part="SUPPLY8" gate="G$1" x="-15.24" y="43.18" rot="R270"/>
+<instance part="GND6" gate="1" x="-91.44" y="109.22"/>
+<instance part="SUPPLY8" gate="G$1" x="-43.18" y="132.08" rot="R270"/>
 <instance part="U2" gate="G$1" x="48.26" y="20.32"/>
 <instance part="GND3" gate="1" x="73.66" y="7.62"/>
@@
 <instance part="PAD2" gate="1" x="129.54" y="66.04" rot="R90"/>
 <instance part="PAD3" gate="1" x="111.76" y="99.06" rot="R180"/>
-<instance part="PAD4" gate="1" x="111.76" y="96.52" rot="R180"/>
+<instance part="PAD4" gate="1" x="111.76" y="91.44" rot="R180"/>
 <instance part="PAD5" gate="1" x="93.98" y="139.7" rot="R180"/>
-<instance part="PAD6" gate="1" x="93.98" y="137.16" rot="R180"/>
+<instance part="PAD6" gate="1" x="93.98" y="132.08" rot="R180"/>
 <instance part="PAD7" gate="1" x="101.6" y="139.7"/>
 <instance part="PAD8" gate="1" x="101.6" y="137.16"/>
@@
 <instance part="SUPPLY9" gate="G$1" x="109.22" y="109.22"/>
 <instance part="GND7" gate="1" x="109.22" y="101.6"/>
-<instance part="PAD11" gate="1" x="-25.4" y="45.72"/>
-<instance part="PAD12" gate="1" x="-25.4" y="43.18"/>
-<instance part="PAD13" gate="1" x="7.62" y="68.58" rot="R90"/>
-<instance part="PAD14" gate="1" x="10.16" y="68.58" rot="R90"/>
+<instance part="PAD11" gate="1" x="-93.98" y="121.92"/>
+<instance part="PAD12" gate="1" x="-96.52" y="132.08"/>
 <instance part="TP2" gate="G$1" x="66.04" y="12.7" rot="R90"/>
 <instance part="TP1" gate="G$1" x="68.58" y="20.32" rot="R90"/>
+<instance part="IC1" gate="G$1" x="-66.04" y="127"/>
+<instance part="R3" gate="G$1" x="-45.72" y="127" rot="R90"/>
+<instance part="R4" gate="G$1" x="-48.26" y="114.3" rot="R90"/>
+<instance part="GND8" gate="1" x="-48.26" y="104.14"/>
+<instance part="C2" gate="G$1" x="-38.1" y="218.44" rot="R90"/>
 </instances>
 <busses>
@@
 <pinref part="C1" gate="G$1" pin="2"/>
 <wire x1="-22.86" y1="208.28" x2="-33.02" y2="203.2" width="0.1524" layer="91"/>
+<pinref part="C2" gate="G$1" pin="2"/>
+<wire x1="-33.02" y1="218.44" x2="-22.86" y2="218.44" width="0.1524" layer="91"/>
+<wire x1="-22.86" y1="218.44" x2="-22.86" y2="208.28" width="0.1524" layer="91"/>
 </segment>
 <segment>
@@
 </segment>
 <segment>
-<pinref part="GND5" gate="1" pin="GND"/>
-<wire x1="10.16" y1="71.12" x2="17.78" y2="71.12" width="0.1524" layer="91"/>
-<wire x1="17.78" y1="71.12" x2="17.78" y2="68.58" width="0.1524" layer="91"/>
-<pinref part="PAD14" gate="1" pin="P"/>
-</segment>
-<segment>
 <pinref part="GND6" gate="1" pin="GND"/>
-<wire x1="-22.86" y1="45.72" x2="-17.78" y2="45.72" width="0.1524" layer="91"/>
+<wire x1="-91.44" y1="121.92" x2="-91.44" y2="111.76" width="0.1524" layer="91"/>
 <pinref part="PAD11" gate="1" pin="P"/>
+<pinref part="IC1" gate="G$1" pin="GND"/>
+<wire x1="-91.44" y1="121.92" x2="-76.2" y2="121.92" width="0.1524" layer="91"/>
 </segment>
 <segment>
@@
 <pinref part="GND7" gate="1" pin="GND"/>
 </segment>
+<segment>
+<pinref part="R4" gate="G$1" pin="1"/>
+<pinref part="GND8" gate="1" pin="GND"/>
+<wire x1="-48.26" y1="106.68" x2="-48.26" y2="109.22" width="0.1524" layer="91"/>
+</segment>
+<segment>
+<wire x1="15.24" y1="78.74" x2="7.62" y2="78.74" width="0.1524" layer="91"/>
+<wire x1="7.62" y1="78.74" x2="7.62" y2="71.12" width="0.1524" layer="91"/>
+<pinref part="IC2" gate="MCU" pin="BOOT0"/>
+<pinref part="GND5" gate="1" pin="GND"/>
+</segment>
 </net>
 <net name="VCC" class="0">
@@
 <pinref part="C1" gate="G$1" pin="1"/>
 <wire x1="-45.72" y1="193.04" x2="-40.64" y2="203.2" width="0.1524" layer="91"/>
+<pinref part="C2" gate="G$1" pin="1"/>
+<wire x1="-40.64" y1="218.44" x2="-53.34" y2="218.44" width="0.1524" layer="91"/>
+<wire x1="-53.34" y1="218.44" x2="-53.34" y2="200.66" width="0.1524" layer="91"/>
 </segment>
 <segment>
@@
 <wire x1="109.22" y1="137.16" x2="104.14" y2="137.16" width="0.1524" layer="91"/>
 <pinref part="PAD8" gate="1" pin="P"/>
-</segment>
-<segment>
-<pinref part="SUPPLY6" gate="G$1" pin="VCC"/>
-<pinref part="R2" gate="G$1" pin="2"/>
-<wire x1="-15.24" y1="73.66" x2="-10.16" y2="73.66" width="0.1524" layer="91"/>
-</segment>
-<segment>
-<pinref part="SUPPLY8" gate="G$1" pin="VCC"/>
-<wire x1="-22.86" y1="43.18" x2="-17.78" y2="43.18" width="0.1524" layer="91"/>
-<pinref part="PAD12" gate="1" pin="P"/>
 </segment>
 <segment>
@@
 <pinref part="SUPPLY9" gate="G$1" pin="VCC"/>
 </segment>
+<segment>
+<pinref part="IC1" gate="G$1" pin="OUT"/>
+<pinref part="SUPPLY8" gate="G$1" pin="VCC"/>
+<pinref part="R3" gate="G$1" pin="2"/>
+<wire x1="-45.72" y1="132.08" x2="-53.34" y2="132.08" width="0.1524" layer="91"/>
+<junction x="-45.72" y="132.08"/>
+</segment>
 </net>
 <net name="N$4" class="0">
@@
 <segment>
 <pinref part="PAD6" gate="1" pin="P"/>
-<wire x1="91.44" y1="137.16" x2="78.74" y2="137.16" width="0.1524" layer="91"/>
-<wire x1="78.74" y1="137.16" x2="78.74" y2="111.76" width="0.1524" layer="91"/>
+<wire x1="91.44" y1="132.08" x2="78.74" y2="132.08" width="0.1524" layer="91"/>
+<wire x1="78.74" y1="132.08" x2="78.74" y2="111.76" width="0.1524" layer="91"/>
 <pinref part="IC2" gate="MCU" pin="PA13"/>
 <wire x1="78.74" y1="111.76" x2="60.96" y2="111.76" width="0.1524" layer="91"/>
@@
 <net name="N$9" class="0">
 <segment>
-<wire x1="60.96" y1="99.06" x2="101.6" y2="99.06" width="0.1524" layer="91"/>
-<wire x1="101.6" y1="99.06" x2="101.6" y2="96.52" width="0.1524" layer="91"/>
-<wire x1="101.6" y1="96.52" x2="109.22" y2="96.52" width="0.1524" layer="91"/>
-<pinref part="IC2" gate="MCU" pin="PA8"/>
+<wire x1="101.6" y1="104.14" x2="101.6" y2="91.44" width="0.1524" layer="91"/>
+<wire x1="101.6" y1="91.44" x2="109.22" y2="91.44" width="0.1524" layer="91"/>
 <pinref part="PAD4" gate="1" pin="P"/>
-</segment>
-</net>
-<net name="N$10" class="0">
-<segment>
-<wire x1="15.24" y1="78.74" x2="7.62" y2="78.74" width="0.1524" layer="91"/>
-<wire x1="7.62" y1="78.74" x2="7.62" y2="73.66" width="0.1524" layer="91"/>
-<pinref part="R2" gate="G$1" pin="1"/>
-<wire x1="7.62" y1="73.66" x2="7.62" y2="71.12" width="0.1524" layer="91"/>
-<wire x1="0" y1="73.66" x2="7.62" y2="73.66" width="0.1524" layer="91"/>
-<pinref part="IC2" gate="MCU" pin="BOOT0"/>
-<pinref part="PAD13" gate="1" pin="P"/>
+<pinref part="IC2" gate="MCU" pin="PA10"/>
+<wire x1="60.96" y1="104.14" x2="101.6" y2="104.14" width="0.1524" layer="91"/>
 </segment>
 </net>
@@
 </segment>
 </net>
+<net name="N$12" class="0">
+<segment>
+<pinref part="IC1" gate="G$1" pin="IN"/>
+<pinref part="PAD12" gate="1" pin="P"/>
+<wire x1="-93.98" y1="132.08" x2="-83.82" y2="132.08" width="0.1524" layer="91"/>
+<pinref part="IC1" gate="G$1" pin="!EN"/>
+<wire x1="-83.82" y1="132.08" x2="-76.2" y2="132.08" width="0.1524" layer="91"/>
+<wire x1="-76.2" y1="127" x2="-83.82" y2="127" width="0.1524" layer="91"/>
+<wire x1="-83.82" y1="127" x2="-83.82" y2="132.08" width="0.1524" layer="91"/>
+<junction x="-83.82" y="132.08"/>
+</segment>
+</net>
+<net name="N$14" class="0">
+<segment>
+<pinref part="IC1" gate="G$1" pin="NC/FB"/>
+<pinref part="R3" gate="G$1" pin="1"/>
+<wire x1="-53.34" y1="121.92" x2="-45.72" y2="121.92" width="0.1524" layer="91"/>
+<pinref part="R4" gate="G$1" pin="2"/>
+<wire x1="-48.26" y1="119.38" x2="-45.72" y2="121.92" width="0.1524" layer="91"/>
+</segment>
+</net>
